Commit message: update small arm base link

File: small_arm_description/urdf/small_arm.xacro (robot description, xacro)
@@ -4,12 +4,12 @@
   <!-- <xacro:include filename="$(find SMW-G02_urdf_description)/urdf/SMW-G02_urdf.trans" />
   <xacro:include filename="$(find SMW-G02_urdf_description)/urdf/SMW-G02_urdf.gazebo" /> -->
-  <xacro:macro name="small_arm" params="parent *origin">
+  <xacro:macro name="small_arm" params="parent base_name:=base_link *origin">
   <joint name="origin_to_base_link" type="fixed">
     <xacro:insert_block name="origin" />
     <parent link="${parent}" />
-    <child link="base_link" />
+    <child link="${base_name}" />
     <axis xyz="0 0 0" />
   </joint>
-  <link name="base_link">
+  <link name="${base_name}">
     <inertial>
       <origin xyz="3.524152480671998e-09 -0.010069634602488222 0.02805569132780735" rpy="0 0 0"/>
@@ -134,5 +134,5 @@
   <joint name="joint1" type="revolute">
     <origin xyz="0.0 0.0 0.053" rpy="0 0 0"/>
-    <parent link="base_link"/>
+    <parent link="${base_name}"/>
     <child link="link1"/>
     <axis xyz="-0.0 0.0 1.0"/>
