Commit message: add gripper on small arm

File: small_arm_description/urdf/small_arm.ros2_control.xacro (robot description, xacro)
@@ -57,4 +57,12 @@
         <state_interface name="effort"/>
       </joint>
+      <joint name="joint7">
+        <param name="id">6</param>
+        <command_interface name="position"/>
+        <command_interface name="velocity"/>
+        <state_interface name="position"/>
+        <state_interface name="velocity"/>
+        <state_interface name="effort"/>
+      </joint>
     </ros2_control>
   </xacro:macro>

File: small_arm_description/urdf/small_arm.xacro (robot description, xacro)
@@ -13,6 +13,6 @@
   <link name="${base_name}">
     <inertial>
-      <origin xyz="3.524152480671998e-09 -0.010069634602488222 0.02805569132780735" rpy="0 0 0"/>
-      <mass value="1.2913743934434603"/>
+      <origin xyz="-0.0002999964758485541 -0.01002821324623266 0.02805569132780727" rpy="0 0 0"/>
+      <mass value="1.29137439344346"/>
       <inertia ixx="0.001017" iyy="0.000798" izz="0.00122" ixy="-0.0" iyz="-3.2e-05" ixz="0.0"/>
     </inertial>
@@ -33,10 +33,10 @@
   <link name="link1">
     <inertial>
-      <origin xyz="0.0005540343927202092 -4.029783931724305e-05 0.03705266234964925" rpy="0 0 0"/>
-      <mass value="0.817001015501461"/>
-      <inertia ixx="0.000382" iyy="0.000409" izz="0.000219" ixy="0.0" iyz="0.0" ixz="-3e-06"/>
-    </inertial>
-    <visual>
-      <origin xyz="-0.0 -0.0 -0.053" rpy="0 0 0"/>
+      <origin xyz="0.0005539067623238434 -2.1382866212631147e-05 0.03707065153568121" rpy="0 0 0"/>
+      <mass value="0.8171892676957183"/>
+      <inertia ixx="0.000382" iyy="0.000408" izz="0.00022" ixy="0.0" iyz="0.0" ixz="-3e-06"/>
+    </inertial>
+    <visual>
+      <origin xyz="0.0003 -4.1e-05 -0.053" rpy="0 0 0"/>
       <geometry>
         <mesh filename="package://small_arm_description/meshes/link_1_1.stl" scale="0.001 0.001 0.001"/>
@@ -45,5 +45,5 @@
     </visual>
     <collision>
-      <origin xyz="-0.0 -0.0 -0.053" rpy="0 0 0"/>
+      <origin xyz="0.0003 -4.1e-05 -0.053" rpy="0 0 0"/>
       <geometry>
         <mesh filename="package://small_arm_description/meshes/link_1_1.stl" scale="0.001 0.001 0.001"/>
@@ -53,10 +53,10 @@
   <link name="link2">
     <inertial>
-      <origin xyz="-0.024402902519636473 -0.0009080265743946556 0.08726119632566089" rpy="0 0 0"/>
-      <mass value="2.2120269627327978"/>
-      <inertia ixx="0.005528" iyy="0.005934" izz="0.001201" ixy="-0.0" iyz="8.5e-05" ixz="-2.5e-05"/>
-    </inertial>
-    <visual>
-      <origin xyz="-0.0245 4.1e-05 -0.109" rpy="0 0 0"/>
+      <origin xyz="-0.024402873741152922 -0.0009180927250929553 0.08726652583609527" rpy="0 0 0"/>
+      <mass value="2.211704028669612"/>
+      <inertia ixx="0.005529" iyy="0.005935" izz="0.001201" ixy="-0.0" iyz="8.6e-05" ixz="-2.5e-05"/>
+    </inertial>
+    <visual>
+      <origin xyz="-0.0242 0.0 -0.109" rpy="0 0 0"/>
       <geometry>
         <mesh filename="package://small_arm_description/meshes/link_2_1.stl" scale="0.001 0.001 0.001"/>
@@ -65,5 +65,5 @@
     </visual>
     <collision>
-      <origin xyz="-0.0245 4.1e-05 -0.109" rpy="0 0 0"/>
+      <origin xyz="-0.0242 0.0 -0.109" rpy="0 0 0"/>
       <geometry>
         <mesh filename="package://small_arm_description/meshes/link_2_1.stl" scale="0.001 0.001 0.001"/>
@@ -73,10 +73,10 @@
   <link name="link3">
     <inertial>
-      <origin xyz="-0.02460877440202336 0.06220285775215952 0.004061931683192799" rpy="0 0 0"/>
-      <mass value="1.4248605431184223"/>
-      <inertia ixx="0.001556" iyy="0.000986" izz="0.001847" ixy="3e-06" iyz="-1.6e-05" ixz="0.0"/>
-    </inertial>
-    <visual>
-      <origin xyz="-0.0244 4.1e-05 -0.264" rpy="0 0 0"/>
+      <origin xyz="-0.024562745448922518 0.06329760185292234 0.004043498969020454" rpy="0 0 0"/>
+      <mass value="1.4560374497113304"/>
+      <inertia ixx="0.001645" iyy="0.001003" izz="0.001935" ixy="2e-06" iyz="-1.2e-05" ixz="-0.0"/>
+    </inertial>
+    <visual>
+      <origin xyz="-0.0241 -0.0 -0.264" rpy="0 0 0"/>
       <geometry>
         <mesh filename="package://small_arm_description/meshes/link_3_1.stl" scale="0.001 0.001 0.001"/>
@@ -85,5 +85,5 @@
     </visual>
     <collision>
-      <origin xyz="-0.0244 4.1e-05 -0.264" rpy="0 0 0"/>
+      <origin xyz="-0.0241 -0.0 -0.264" rpy="0 0 0"/>
       <geometry>
         <mesh filename="package://small_arm_description/meshes/link_3_1.stl" scale="0.001 0.001 0.001"/>
@@ -93,10 +93,10 @@
   <link name="link4">
     <inertial>
-      <origin xyz="0.0001935598278808653 0.028814811744396554 -1.4041829764444014e-05" rpy="0 0 0"/>
-      <mass value="0.44007071116462465"/>
-      <inertia ixx="0.000141" iyy="8.2e-05" izz="0.000139" ixy="-1e-06" iyz="0.0" ixz="-0.0"/>
-    </inertial>
-    <visual>
-      <origin xyz="0.0003 -0.100725 -0.265316" rpy="0 0 0"/>
+      <origin xyz="-0.0001915907936059267 0.028749765366266278 1.3933167071766839e-05" rpy="0 0 0"/>
+      <mass value="0.4445934457308041"/>
+      <inertia ixx="0.000143" iyy="8.2e-05" izz="0.00014" ixy="1e-06" iyz="-0.0" ixz="-0.0"/>
+    </inertial>
+    <visual>
+      <origin xyz="0.0006 -0.100766 -0.265316" rpy="0 0 0"/>
       <geometry>
         <mesh filename="package://small_arm_description/meshes/link_4_1.stl" scale="0.001 0.001 0.001"/>
@@ -105,5 +105,5 @@
     </visual>
     <collision>
-      <origin xyz="0.0003 -0.100725 -0.265316" rpy="0 0 0"/>
+      <origin xyz="0.0006 -0.100766 -0.265316" rpy="0 0 0"/>
       <geometry>
         <mesh filename="package://small_arm_description/meshes/link_4_1.stl" scale="0.001 0.001 0.001"/>
@@ -113,10 +113,10 @@
   <link name="link5">
     <inertial>
-      <origin xyz="-0.019050063908979883 0.006974684180871771 -0.04469598937792321" rpy="0 0 0"/>
-      <mass value="0.6811318961965678"/>
-      <inertia ixx="0.000369" iyy="0.000349" izz="0.000252" ixy="-0.0" iyz="1.6e-05" ixz="0.0"/>
-    </inertial>
-    <visual>
-      <origin xyz="-0.0197 -0.144606 -0.265316" rpy="0 0 0"/>
+      <origin xyz="-0.019004907946417172 0.007238676029536678 -0.043336314243680424" rpy="0 0 0"/>
+      <mass value="0.970501435691462"/>
+      <inertia ixx="0.00064" iyy="0.000557" izz="0.000514" ixy="-1e-06" iyz="-1.4e-05" ixz="-0.0"/>
+    </inertial>
+    <visual>
+      <origin xyz="-0.0174 -0.144647 -0.265316" rpy="0 0 0"/>
       <geometry>
         <mesh filename="package://small_arm_description/meshes/link_5_1.stl" scale="0.001 0.001 0.001"/>
@@ -125,5 +125,5 @@
     </visual>
     <collision>
-      <origin xyz="-0.0197 -0.144606 -0.265316" rpy="0 0 0"/>
+      <origin xyz="-0.0174 -0.144647 -0.265316" rpy="0 0 0"/>
       <geometry>
         <mesh filename="package://small_arm_description/meshes/link_5_1.stl" scale="0.001 0.001 0.001"/>
@@ -131,10 +131,89 @@
     </collision>
   </link>
-  <link name="link6"/>
+  <link name="link6">
+    <inertial>
+      <origin xyz="-5.506012312750386e-15 4.949917709884399e-07 -0.0026212148467256724" rpy="0 0 0"/>
+      <mass value="0.025512046719187297"/>
+      <inertia ixx="2e-06" iyy="2e-06" izz="4e-06" ixy="0.0" iyz="0.0" ixz="-0.0"/>
+    </inertial>
+    <visual>
+      <origin xyz="0.0016 -0.144647 -0.196297" rpy="0 0 0"/>
+      <geometry>
+        <mesh filename="package://small_arm_description/meshes/link_6_1.stl" scale="0.001 0.001 0.001"/>
+      </geometry>
+      <material name="silver"/>
+    </visual>
+    <collision>
+      <origin xyz="0.0016 -0.144647 -0.196297" rpy="0 0 0"/>
+      <geometry>
+        <mesh filename="package://small_arm_description/meshes/link_6_1.stl" scale="0.001 0.001 0.001"/>
+      </geometry>
+    </collision>
+  </link>
+  <link name="gripper_link1">
+    <inertial>
+      <origin xyz="0.009922614801186412 -0.01909950500842314 -0.024668286066997724" rpy="0 0 0"/>
+      <mass value="0.16533614239781452"/>
+      <inertia ixx="0.000142" iyy="7.7e-05" izz="8.2e-05" ixy="-0.0" iyz="-0.0" ixz="5e-06"/>
+    </inertial>
+    <visual>
+      <origin xyz="-0.0204 -0.163647 -0.169647" rpy="0 0 0"/>
+      <geometry>
+        <mesh filename="package://small_arm_description/meshes/Craw_2_1.stl" scale="0.001 0.001 0.001"/>
+      </geometry>
+      <material name="silver"/>
+    </visual>
+    <collision>
+      <origin xyz="-0.0204 -0.163647 -0.169647" rpy="0 0 0"/>
+      <geometry>
+        <mesh filename="package://small_arm_description/meshes/Craw_2_1.stl" scale="0.001 0.001 0.001"/>
+      </geometry>
+    </collision>
+  </link>
+<link name="gripper_link2">
+  <inertial>
+    <origin xyz="-0.004639846314339198 0.0002472053469017299 -0.02547670727420101" rpy="0 0 0"/>
+    <mass value="0.6910133017831432"/>
+    <inertia ixx="0.000328" iyy="0.000563" izz="0.000489" ixy="-3e-06" iyz="-1e-06" ixz="-0.000126"/>
+  </inertial>
+  <visual>
+    <origin xyz="0.0016 -0.144647 -0.190797" rpy="0 0 0"/>
+    <geometry>
+      <mesh filename="package://small_arm_description/meshes/Craw_1_1.stl" scale="0.001 0.001 0.001"/>
+    </geometry>
+    <material name="silver"/>
+  </visual>
+  <collision>
+    <origin xyz="0.0016 -0.144647 -0.190797" rpy="0 0 0"/>
+    <geometry>
+      <mesh filename="package://small_arm_description/meshes/Craw_1_1.stl" scale="0.001 0.001 0.001"/>
+    </geometry>
+  </collision>
+</link>
+  <link name="camera_link">
+    <inertial>
+      <origin xyz="-0.02250186173818042 -4.850013210841442e-05 -0.012169837419761076" rpy="0 0 0"/>
+      <mass value="0.3783798760930688"/>
+      <inertia ixx="3.5e-05" iyy="0.00024" izz="0.000238" ixy="-0.0" iyz="-0.0" ixz="0.0"/>
+    </inertial>
+    <visual>
+      <origin xyz="-0.0209 -0.194439 -0.219247" rpy="0 0 0"/>
+      <geometry>
+        <mesh filename="package://small_arm_description/meshes/RealSence_1.stl" scale="0.001 0.001 0.001"/>
+      </geometry>
+      <material name="silver"/>
+    </visual>
+    <collision>
+      <origin xyz="-0.0209 -0.194439 -0.219247" rpy="0 0 0"/>
+      <geometry>
+        <mesh filename="package://small_arm_description/meshes/RealSence_1.stl" scale="0.001 0.001 0.001"/>
+      </geometry>
+    </collision>
+  </link>
   <joint name="joint1" type="revolute">
-    <origin xyz="0.0 0.0 0.053" rpy="0 0 0"/>
+    <origin xyz="-0.0003 4.1e-05 0.053" rpy="0 0 0"/>
     <parent link="${base_name}"/>
     <child link="link1"/>
-    <axis xyz="-0.0 0.0 1.0"/>
+    <axis xyz="-0.0 -0.0 1.0"/>
     <limit
       lower="-3.14"
@@ -158,5 +237,5 @@
     <parent link="link2"/>
     <child link="link3"/>
-    <axis xyz="-1.0 -0.0 -0.0"/>
+    <axis xyz="1.0 0.0 0.0"/>
     <limit
       lower="-3.14"
@@ -177,8 +256,8 @@
   </joint>
   <joint name="joint5" type="revolute">
-    <origin xyz="0.02 0.043881 0.0" rpy="0 0 0"/>
+    <origin xyz="0.018 0.043881 0.0" rpy="0 0 0"/>
     <parent link="link4"/>
     <child link="link5"/>
-    <axis xyz="1.0 -0.0 -0.0"/>
+    <axis xyz="1.0 0.0 -0.0"/>
     <limit
       lower="-3.14"
@@ -188,13 +267,34 @@
   </joint>
   <joint name="joint6" type="revolute">
-    <origin xyz="0.02 0.043881 0.0" rpy="0 0 0"/>
+    <origin xyz="-0.019 0.0 -0.069019" rpy="0 0 0"/>
     <parent link="link5"/>
     <child link="link6"/>
-    <axis xyz="1.0 -0.0 -0.0"/>
-    <limit
-      lower="-3.14"
-      upper="3.14"
-      effort="1"
-      velocity="4.8" />
+    <axis xyz="0.0 -0.0 -1.0"/>
+    <limit
+      lower="-3.14"
+      upper="3.14"
+      effort="1"
+      velocity="4.8" />
+  </joint>
+  <joint name="joint7" type="revolute">
+    <origin xyz="0.022 0.019 -0.02115" rpy="0 0 0"/>
+    <parent link="gripper_link2"/>
+    <child link="gripper_link1"/>
+    <axis xyz="0.0 1.0 0.0"/>
+    <limit
+      lower="-3.14"
+      upper="3.14"
+      effort="1"
+      velocity="4.8" />
+  </joint>
+  <joint name="girpper_fixed" type="fixed">
+    <origin xyz="0.0 0.0 -0.0055" rpy="0 0 0"/>
+    <parent link="link6"/>
+    <child link="gripper_link2"/>
+  </joint>
+  <joint name="camera_fixed" type="fixed">
+    <origin xyz="0.0035 0.049792 -0.046069" rpy="0 0 0"/>
+    <parent link="link5"/>
+    <child link="camera_link"/>
   </joint>
   </xacro:macro>

File: small_arm_moveit_config/config/small_arm.ros2_control.xacro (robot description, xacro)
@@ -1,10 +1,17 @@
 <?xml version="1.0"?>
 <robot xmlns:xacro="http://www.ros.org/wiki/xacro">
-    <xacro:macro name="small_arm_ros2_control" params="name initial_positions_file">
+    <xacro:macro name="small_arm_ros2_control" params="name initial_positions_file ros2_control_hardware_type">
         <xacro:property name="initial_positions" value="${load_yaml(initial_positions_file)['initial_positions']}"/>
         <ros2_control name="${name}" type="system">
             <hardware>
-                <!-- By default, set up controllers for simulation. This won't work on real hardware -->
-                <plugin>mock_components/GenericSystem</plugin>
+                <xacro:if value="${ros2_control_hardware_type == 'fake'}">
+                    <plugin>mock_components/GenericSystem</plugin>
+                </xacro:if>
+                <xacro:if value="${ros2_control_hardware_type == 'real'}">
+                    <plugin>dynamixel_hardware/DynamixelHardware</plugin>
+                    <param name="usb_port">/dev/ttyUSB0</param>
+                    <param name="baud_rate">115200</param>
+                    <param name="use_dummy">false</param>
+                </xacro:if>
             </hardware>
             <joint name="joint1">

File: small_arm_moveit_config/config/small_arm.urdf.xacro (robot description, xacro)
@@ -2,8 +2,9 @@
 <robot xmlns:xacro="http://www.ros.org/wiki/xacro" name="small_arm">
     <xacro:arg name="initial_positions_file" default="initial_positions.yaml" />
+    <xacro:arg name="ros2_control_hardware_type" default="mock_components" />
     <!-- Import small_arm urdf file -->
     <xacro:include filename="$(find small_arm_description)/urdf/small_arm.urdf.xacro" />
     <!-- Import control_xacro -->
     <xacro:include filename="small_arm.ros2_control.xacro" />
-    <xacro:small_arm_ros2_control name="FakeSystem" initial_positions_file="$(arg initial_positions_file)"/>
+    <xacro:small_arm_ros2_control name="FakeSystem" initial_positions_file="$(arg initial_positions_file)" ros2_control_hardware_type="$(arg ros2_control_hardware_type)"/>
 </robot>

Commit message: update real robot info

File: small_arm_description/urdf/small_arm.ros2_control.xacro (robot description, xacro)
@@ -7,5 +7,5 @@
         <param name="usb_port">/dev/ttyUSB0</param>
         <param name="baud_rate">115200</param>
-        <param name="use_dummy">true</param>
+        <param name="use_dummy">false</param>
       </hardware>
       <joint name="joint1">
@@ -58,5 +58,5 @@
       </joint>
       <joint name="joint7">
-        <param name="id">6</param>
+        <param name="id">7</param>
         <command_interface name="position"/>
         <command_interface name="velocity"/>

File: small_arm_moveit_config/config/small_arm.ros2_control.xacro (robot description, xacro)
@@ -16,4 +16,5 @@
             </hardware>
             <joint name="joint1">
+            <param name="id">1</param>
                 <command_interface name="position"/>
                 <state_interface name="position">
@@ -23,4 +24,5 @@
             </joint>
             <joint name="joint2">
+            <param name="id">2</param>
                 <command_interface name="position"/>
                 <state_interface name="position">
@@ -30,4 +32,5 @@
             </joint>
             <joint name="joint3">
+            <param name="id">3</param>
                 <command_interface name="position"/>
                 <state_interface name="position">
@@ -37,4 +40,5 @@
             </joint>
             <joint name="joint4">
+            <param name="id">4</param>
                 <command_interface name="position"/>
                 <state_interface name="position">
@@ -44,4 +48,5 @@
             </joint>
             <joint name="joint5">
+            <param name="id">5</param>
                 <command_interface name="position"/>
                 <state_interface name="position">
@@ -51,4 +56,5 @@
             </joint>
             <joint name="joint6">
+            <param name="id">6</param>
                 <command_interface name="position"/>
                 <state_interface name="position">
@@ -57,4 +63,12 @@
                 <state_interface name="velocity"/>
             </joint>
+            <joint name="joint7">
+            <param name="id">7</param>
+                <command_interface name="position"/>
+                <state_interface name="position">
+                  <param name="initial_value">${initial_positions['joint7']}</param>
+                </state_interface>
+                <state_interface name="velocity"/>
+            </joint>
         </ros2_control>
     </xacro:macro>
