Commit message: modfiy small arm gripper

File: small_arm_description/urdf/small_arm.ros2_control.xacro (robot description, xacro)
@@ -57,5 +57,5 @@
         <state_interface name="effort"/>
       </joint>
-      <joint name="joint7">
+      <joint name="gripper_joint1">
         <param name="id">7</param>
         <command_interface name="position"/>
@@ -65,4 +65,16 @@
         <state_interface name="effort"/>
       </joint>
+      <!-- <hardware>
+          <plugin>fake_components/GenericSystem</plugin>
+      </hardware>
+      <joint name="gripper_joint2">
+        <param name="mimic">gripper_joint1</param>
+        <param name="multiplier">-1</param>
+        <command_interface name="position"/>
+        <command_interface name="velocity"/>
+        <state_interface name="position"/>
+        <state_interface name="velocity"/>
+        <state_interface name="effort"/>
+      </joint> -->
     </ros2_control>
   </xacro:macro>

File: small_arm_description/urdf/small_arm.xacro (robot description, xacro)
@@ -13,5 +13,5 @@
   <link name="${base_name}">
     <inertial>
-      <origin xyz="-0.0002999964758485541 -0.01002821324623266 0.02805569132780727" rpy="0 0 0"/>
+      <origin xyz="3.5241524236579847e-09 -0.010028213246232836 0.028055691327807355" rpy="0 0 0"/>
       <mass value="1.29137439344346"/>
       <inertia ixx="0.001017" iyy="0.000798" izz="0.00122" ixy="-0.0" iyz="-3.2e-05" ixz="0.0"/>
@@ -33,10 +33,10 @@
   <link name="link1">
     <inertial>
-      <origin xyz="0.0005539067623238434 -2.1382866212631147e-05 0.03707065153568121" rpy="0 0 0"/>
-      <mass value="0.8171892676957183"/>
-      <inertia ixx="0.000382" iyy="0.000408" izz="0.00022" ixy="0.0" iyz="0.0" ixz="-3e-06"/>
-    </inertial>
-    <visual>
-      <origin xyz="0.0003 -4.1e-05 -0.053" rpy="0 0 0"/>
+      <origin xyz="0.0005540343927201894 -3.987648307993698e-05 0.03705266234964923" rpy="0 0 0"/>
+      <mass value="0.8170010155014609"/>
+      <inertia ixx="0.000382" iyy="0.000409" izz="0.000219" ixy="0.0" iyz="0.0" ixz="-3e-06"/>
+    </inertial>
+    <visual>
+      <origin xyz="0.0 -4.1e-05 -0.053" rpy="0 0 0"/>
       <geometry>
         <mesh filename="package://small_arm_description/meshes/link_1_1.stl" scale="0.001 0.001 0.001"/>
@@ -45,5 +45,5 @@
     </visual>
     <collision>
-      <origin xyz="0.0003 -4.1e-05 -0.053" rpy="0 0 0"/>
+      <origin xyz="0.0 -4.1e-05 -0.053" rpy="0 0 0"/>
       <geometry>
         <mesh filename="package://small_arm_description/meshes/link_1_1.stl" scale="0.001 0.001 0.001"/>
@@ -53,10 +53,10 @@
   <link name="link2">
     <inertial>
-      <origin xyz="-0.024402873741152922 -0.0009180927250929553 0.08726652583609527" rpy="0 0 0"/>
-      <mass value="2.211704028669612"/>
-      <inertia ixx="0.005529" iyy="0.005935" izz="0.001201" ixy="-0.0" iyz="8.6e-05" ixz="-2.5e-05"/>
-    </inertial>
-    <visual>
-      <origin xyz="-0.0242 0.0 -0.109" rpy="0 0 0"/>
+      <origin xyz="-0.024402503506776505 -0.000948414974992276 0.08721596254239226" rpy="0 0 0"/>
+      <mass value="2.207557884875517"/>
+      <inertia ixx="0.005523" iyy="0.005928" izz="0.001196" ixy="-0.0" iyz="8.7e-05" ixz="-2.5e-05"/>
+    </inertial>
+    <visual>
+      <origin xyz="-0.0245 0.0 -0.109" rpy="0 0 0"/>
       <geometry>
         <mesh filename="package://small_arm_description/meshes/link_2_1.stl" scale="0.001 0.001 0.001"/>
@@ -65,5 +65,5 @@
     </visual>
     <collision>
-      <origin xyz="-0.0242 0.0 -0.109" rpy="0 0 0"/>
+      <origin xyz="-0.0245 0.0 -0.109" rpy="0 0 0"/>
       <geometry>
         <mesh filename="package://small_arm_description/meshes/link_2_1.stl" scale="0.001 0.001 0.001"/>
@@ -73,10 +73,10 @@
   <link name="link3">
     <inertial>
-      <origin xyz="-0.024562745448922518 0.06329760185292234 0.004043498969020454" rpy="0 0 0"/>
-      <mass value="1.4560374497113304"/>
-      <inertia ixx="0.001645" iyy="0.001003" izz="0.001935" ixy="2e-06" iyz="-1.2e-05" ixz="-0.0"/>
-    </inertial>
-    <visual>
-      <origin xyz="-0.0241 -0.0 -0.264" rpy="0 0 0"/>
+      <origin xyz="-0.024604835871039465 0.06321426100068431 0.0039992416943318565" rpy="0 0 0"/>
+      <mass value="1.4545470633400195"/>
+      <inertia ixx="0.001649" iyy="0.001003" izz="0.00194" ixy="2e-06" iyz="-1.2e-05" ixz="0.0"/>
+    </inertial>
+    <visual>
+      <origin xyz="-0.0244 -0.0 -0.264" rpy="0 0 0"/>
       <geometry>
         <mesh filename="package://small_arm_description/meshes/link_3_1.stl" scale="0.001 0.001 0.001"/>
@@ -85,5 +85,5 @@
     </visual>
     <collision>
-      <origin xyz="-0.0241 -0.0 -0.264" rpy="0 0 0"/>
+      <origin xyz="-0.0244 -0.0 -0.264" rpy="0 0 0"/>
       <geometry>
         <mesh filename="package://small_arm_description/meshes/link_3_1.stl" scale="0.001 0.001 0.001"/>
@@ -93,10 +93,10 @@
   <link name="link4">
     <inertial>
-      <origin xyz="-0.0001915907936059267 0.028749765366266278 1.3933167071766839e-05" rpy="0 0 0"/>
-      <mass value="0.4445934457308041"/>
-      <inertia ixx="0.000143" iyy="8.2e-05" izz="0.00014" ixy="1e-06" iyz="-0.0" ixz="-0.0"/>
-    </inertial>
-    <visual>
-      <origin xyz="0.0006 -0.100766 -0.265316" rpy="0 0 0"/>
+      <origin xyz="0.0005772929478554495 0.02874769471007499 0.00014670041370268283" rpy="0 0 0"/>
+      <mass value="0.4457408919666805"/>
+      <inertia ixx="0.000144" iyy="8.2e-05" izz="0.00014" ixy="-1e-06" iyz="-0.0" ixz="-0.0"/>
+    </inertial>
+    <visual>
+      <origin xyz="0.0003 -0.100766 -0.265316" rpy="0 0 0"/>
       <geometry>
         <mesh filename="package://small_arm_description/meshes/link_4_1.stl" scale="0.001 0.001 0.001"/>
@@ -105,5 +105,5 @@
     </visual>
     <collision>
-      <origin xyz="0.0006 -0.100766 -0.265316" rpy="0 0 0"/>
+      <origin xyz="0.0003 -0.100766 -0.265316" rpy="0 0 0"/>
       <geometry>
         <mesh filename="package://small_arm_description/meshes/link_4_1.stl" scale="0.001 0.001 0.001"/>
@@ -113,10 +113,10 @@
   <link name="link5">
     <inertial>
-      <origin xyz="-0.019004907946417172 0.007238676029536678 -0.043336314243680424" rpy="0 0 0"/>
-      <mass value="0.970501435691462"/>
-      <inertia ixx="0.00064" iyy="0.000557" izz="0.000514" ixy="-1e-06" iyz="-1.4e-05" ixz="-0.0"/>
-    </inertial>
-    <visual>
-      <origin xyz="-0.0174 -0.144647 -0.265316" rpy="0 0 0"/>
+      <origin xyz="-0.019082924173376172 0.006958151104480087 -0.04482191950153944" rpy="0 0 0"/>
+      <mass value="0.9868678983343436"/>
+      <inertia ixx="0.000651" iyy="0.000558" izz="0.000526" ixy="0.0" iyz="-1.2e-05" ixz="0.0"/>
+    </inertial>
+    <visual>
+      <origin xyz="-0.0187 -0.144647 -0.265441" rpy="0 0 0"/>
       <geometry>
         <mesh filename="package://small_arm_description/meshes/link_5_1.stl" scale="0.001 0.001 0.001"/>
@@ -125,5 +125,5 @@
     </visual>
     <collision>
-      <origin xyz="-0.0174 -0.144647 -0.265316" rpy="0 0 0"/>
+      <origin xyz="-0.0187 -0.144647 -0.265441" rpy="0 0 0"/>
       <geometry>
         <mesh filename="package://small_arm_description/meshes/link_5_1.stl" scale="0.001 0.001 0.001"/>
@@ -133,19 +133,19 @@
   <link name="link6">
     <inertial>
-      <origin xyz="-5.506012312750386e-15 4.949917709884399e-07 -0.0026212148467256724" rpy="0 0 0"/>
-      <mass value="0.025512046719187297"/>
-      <inertia ixx="2e-06" iyy="2e-06" izz="4e-06" ixy="0.0" iyz="0.0" ixz="-0.0"/>
-    </inertial>
-    <visual>
-      <origin xyz="0.0016 -0.144647 -0.196297" rpy="0 0 0"/>
-      <geometry>
-        <mesh filename="package://small_arm_description/meshes/link_6_1.stl" scale="0.001 0.001 0.001"/>
-      </geometry>
-      <material name="silver"/>
-    </visual>
-    <collision>
-      <origin xyz="0.0016 -0.144647 -0.196297" rpy="0 0 0"/>
-      <geometry>
-        <mesh filename="package://small_arm_description/meshes/link_6_1.stl" scale="0.001 0.001 0.001"/>
+      <origin xyz="0.004698639386755362 0.0003750363685992575 -0.018998646992087587" rpy="0 0 0"/>
+      <mass value="0.5087647252977904"/>
+      <inertia ixx="9.4e-05" iyy="0.000223" izz="0.000231" ixy="-1e-06" iyz="0.0" ixz="1e-06"/>
+    </inertial>
+    <visual>
+      <origin xyz="0.0004 -0.144647 -0.190922" rpy="0 0 0"/>
+      <geometry>
+        <mesh filename="package://small_arm_description/meshes/Claw_base_1.stl" scale="0.001 0.001 0.001"/>
+      </geometry>
+      <material name="silver"/>
+    </visual>
+    <collision>
+      <origin xyz="0.0004 -0.144647 -0.190922" rpy="0 0 0"/>
+      <geometry>
+        <mesh filename="package://small_arm_description/meshes/Claw_base_1.stl" scale="0.001 0.001 0.001"/>
       </geometry>
     </collision>
@@ -153,64 +153,64 @@
   <link name="gripper_link1">
     <inertial>
-      <origin xyz="0.009922614801186412 -0.01909950500842314 -0.024668286066997724" rpy="0 0 0"/>
-      <mass value="0.16533614239781452"/>
-      <inertia ixx="0.000142" iyy="7.7e-05" izz="8.2e-05" ixy="-0.0" iyz="-0.0" ixz="5e-06"/>
-    </inertial>
-    <visual>
-      <origin xyz="-0.0204 -0.163647 -0.169647" rpy="0 0 0"/>
-      <geometry>
-        <mesh filename="package://small_arm_description/meshes/Craw_2_1.stl" scale="0.001 0.001 0.001"/>
-      </geometry>
-      <material name="silver"/>
-    </visual>
-    <collision>
-      <origin xyz="-0.0204 -0.163647 -0.169647" rpy="0 0 0"/>
-      <geometry>
-        <mesh filename="package://small_arm_description/meshes/Craw_2_1.stl" scale="0.001 0.001 0.001"/>
+      <origin xyz="0.008617592547608088 -0.019099487462018033 -0.018966140525552982" rpy="0 0 0"/>
+      <mass value="0.27120735685123026"/>
+      <inertia ixx="0.000219" iyy="0.000142" izz="0.000135" ixy="0.0" iyz="-0.0" ixz="2e-05"/>
+    </inertial>
+    <visual>
+      <origin xyz="-0.0216 -0.163647 -0.169772" rpy="0 0 0"/>
+      <geometry>
+        <mesh filename="package://small_arm_description/meshes/Claw_1_1.stl" scale="0.001 0.001 0.001"/>
+      </geometry>
+      <material name="silver"/>
+    </visual>
+    <collision>
+      <origin xyz="-0.0216 -0.163647 -0.169772" rpy="0 0 0"/>
+      <geometry>
+        <mesh filename="package://small_arm_description/meshes/Claw_1_1.stl" scale="0.001 0.001 0.001"/>
       </geometry>
     </collision>
   </link>
 <link name="gripper_link2">
-  <inertial>
-    <origin xyz="-0.004639846314339198 0.0002472053469017299 -0.02547670727420101" rpy="0 0 0"/>
-    <mass value="0.6910133017831432"/>
-    <inertia ixx="0.000328" iyy="0.000563" izz="0.000489" ixy="-3e-06" iyz="-1e-06" ixz="-0.000126"/>
-  </inertial>
-  <visual>
-    <origin xyz="0.0016 -0.144647 -0.190797" rpy="0 0 0"/>
-    <geometry>
-      <mesh filename="package://small_arm_description/meshes/Craw_1_1.stl" scale="0.001 0.001 0.001"/>
-    </geometry>
-    <material name="silver"/>
-  </visual>
-  <collision>
-    <origin xyz="0.0016 -0.144647 -0.190797" rpy="0 0 0"/>
-    <geometry>
-      <mesh filename="package://small_arm_description/meshes/Craw_1_1.stl" scale="0.001 0.001 0.001"/>
-    </geometry>
-  </collision>
-</link>
+    <inertial>
+      <origin xyz="-0.0077905784072223 -0.019078107759134433 -0.01729592412140632" rpy="0 0 0"/>
+      <mass value="0.2862239344986947"/>
+      <inertia ixx="0.000234" iyy="0.00015" izz="0.000143" ixy="0.0" iyz="0.0" ixz="-2.3e-05"/>
+    </inertial>
+    <visual>
+      <origin xyz="0.0224 -0.163582 -0.169772" rpy="0 0 0"/>
+      <geometry>
+        <mesh filename="package://small_arm_description/meshes/Claw_2_1.stl" scale="0.001 0.001 0.001"/>
+      </geometry>
+      <material name="silver"/>
+    </visual>
+    <collision>
+      <origin xyz="0.0224 -0.163582 -0.169772" rpy="0 0 0"/>
+      <geometry>
+        <mesh filename="package://small_arm_description/meshes/Claw_2_1.stl" scale="0.001 0.001 0.001"/>
+      </geometry>
+    </collision>
+  </link>
   <link name="camera_link">
     <inertial>
-      <origin xyz="-0.02250186173818042 -4.850013210841442e-05 -0.012169837419761076" rpy="0 0 0"/>
-      <mass value="0.3783798760930688"/>
+      <origin xyz="-1.8617389460899472e-06 -0.008048500132108033 -0.012169837419856416" rpy="0 0 0"/>
+      <mass value="0.3783798760930714"/>
       <inertia ixx="3.5e-05" iyy="0.00024" izz="0.000238" ixy="-0.0" iyz="-0.0" ixz="0.0"/>
     </inertial>
     <visual>
-      <origin xyz="-0.0209 -0.194439 -0.219247" rpy="0 0 0"/>
-      <geometry>
-        <mesh filename="package://small_arm_description/meshes/RealSence_1.stl" scale="0.001 0.001 0.001"/>
-      </geometry>
-      <material name="silver"/>
-    </visual>
-    <collision>
-      <origin xyz="-0.0209 -0.194439 -0.219247" rpy="0 0 0"/>
-      <geometry>
-        <mesh filename="package://small_arm_description/meshes/RealSence_1.stl" scale="0.001 0.001 0.001"/>
+      <origin xyz="0.0004 -0.202439 -0.219372" rpy="0 0 0"/>
+      <geometry>
+        <mesh filename="package://small_arm_description/meshes/Camera_1.stl" scale="0.001 0.001 0.001"/>
+      </geometry>
+      <material name="silver"/>
+    </visual>
+    <collision>
+      <origin xyz="0.0004 -0.202439 -0.219372" rpy="0 0 0"/>
+      <geometry>
+        <mesh filename="package://small_arm_description/meshes/Camera_1.stl" scale="0.001 0.001 0.001"/>
       </geometry>
     </collision>
   </link>
   <joint name="joint1" type="revolute">
-    <origin xyz="-0.0003 4.1e-05 0.053" rpy="0 0 0"/>
+    <origin xyz="0.0 4.1e-05 0.053" rpy="0 0 0"/>
     <parent link="${base_name}"/>
     <child link="link1"/>
@@ -256,5 +256,5 @@
   </joint>
   <joint name="joint5" type="revolute">
-    <origin xyz="0.018 0.043881 0.0" rpy="0 0 0"/>
+    <origin xyz="0.019 0.043881 0.000125" rpy="0 0 0"/>
     <parent link="link4"/>
     <child link="link5"/>
@@ -277,7 +277,7 @@
       velocity="4.8" />
   </joint>
-  <joint name="joint7" type="revolute">
+  <joint name="gripper_joint1" type="revolute">
     <origin xyz="0.022 0.019 -0.02115" rpy="0 0 0"/>
-    <parent link="gripper_link2"/>
+    <parent link="link6"/>
     <child link="gripper_link1"/>
     <axis xyz="0.0 1.0 0.0"/>
@@ -288,11 +288,23 @@
       velocity="4.8" />
   </joint>
-  <joint name="girpper_fixed" type="fixed">
+  <joint name="gripper_joint2" type="continuous">
+    <origin xyz="-0.022 0.018935 -0.02115" rpy="0 0 0"/>
+    <parent link="link6"/>
+    <child link="gripper_link2"/>
+    <axis xyz="-0.0 1.0 -0.0"/>
+    <mimic joint="gripper_joint1" multiplier="-1"/>
+    <!-- <limit
+      lower="-3.14"
+      upper="3.14"
+      effort="1"
+      velocity="4.8" /> -->
+  </joint>
+  <!-- <joint name="girpper_fixed" type="fixed">
     <origin xyz="0.0 0.0 -0.0055" rpy="0 0 0"/>
     <parent link="link6"/>
-    <child link="gripper_link2"/>
-  </joint>
+    <child link="gripper_link1"/>
+  </joint> -->
   <joint name="camera_fixed" type="fixed">
-    <origin xyz="0.0035 0.049792 -0.046069" rpy="0 0 0"/>
+    <origin xyz="-0.0191 0.057792 -0.046069" rpy="0 0 0"/>
     <parent link="link5"/>
     <child link="camera_link"/>

File: small_arm_moveit_config/config/small_arm.ros2_control.xacro (robot description, xacro)
@@ -63,5 +63,5 @@
         <state_interface name="effort"/>
       </joint>
-      <joint name="joint7">
+      <joint name="gripper_joint1">
         <param name="id">7</param>
         <command_interface name="position"/>
@@ -71,57 +71,10 @@
         <state_interface name="effort"/>
       </joint>
-            <!-- <joint name="joint1">
-            <param name="id">1</param>
+            <!-- <joint name="gripper_joint2">
+                <param name="mimic">gripper_joint1</param>
+                <param name="multiplier">-1</param>
                 <command_interface name="position"/>
                 <state_interface name="position">
-                  <param name="initial_value">${initial_positions['joint1']}</param>
-                </state_interface>
-                <state_interface name="velocity"/>
-            </joint>
-            <joint name="joint2">
-            <param name="id">2</param>
-                <command_interface name="position"/>
-                <state_interface name="position">
-                  <param name="initial_value">${initial_positions['joint2']}</param>
-                </state_interface>
-                <state_interface name="velocity"/>
-            </joint>
-            <joint name="joint3">
-            <param name="id">3</param>
-                <command_interface name="position"/>
-                <state_interface name="position">
-                  <param name="initial_value">${initial_positions['joint3']}</param>
-                </state_interface>
-                <state_interface name="velocity"/>
-            </joint>
-            <joint name="joint4">
-            <param name="id">4</param>
-                <command_interface name="position"/>
-                <state_interface name="position">
-                  <param name="initial_value">${initial_positions['joint4']}</param>
-                </state_interface>
-                <state_interface name="velocity"/>
-            </joint>
-            <joint name="joint5">
-            <param name="id">5</param>
-                <command_interface name="position"/>
-                <state_interface name="position">
-                  <param name="initial_value">${initial_positions['joint5']}</param>
-                </state_interface>
-                <state_interface name="velocity"/>
-            </joint>
-            <joint name="joint6">
-            <param name="id">6</param>
-                <command_interface name="position"/>
-                <state_interface name="position">
-                  <param name="initial_value">${initial_positions['joint6']}</param>
-                </state_interface>
-                <state_interface name="velocity"/>
-            </joint>
-            <joint name="joint7">
-            <param name="id">7</param>
-                <command_interface name="position"/>
-                <state_interface name="position">
-                  <param name="initial_value">${initial_positions['joint7']}</param>
+                  <param name="initial_value">${initial_positions['gripper_joint1']}</param>
                 </state_interface>
                 <state_interface name="velocity"/>

File: small_arm_moveit_config/config/small_arm.urdf.xacro (robot description, xacro)
@@ -2,5 +2,5 @@
 <robot xmlns:xacro="http://www.ros.org/wiki/xacro" name="small_arm">
     <xacro:arg name="initial_positions_file" default="initial_positions.yaml" />
-    <xacro:arg name="ros2_control_hardware_type" default="mock_components" />
+    <xacro:arg name="ros2_control_hardware_type" default="fake" />
     <!-- Import small_arm urdf file -->
     <xacro:include filename="$(find small_arm_description)/urdf/small_arm.urdf.xacro" />
