Commit message: new version of small arm

File: small_arm_description/urdf/small_arm copy 2.xacro (robot description, xacro)
@@ -12,19 +12,19 @@
   </joint>
   <link name="${base_name}">
-  <inertial>
-    <origin xyz="6.583680213469905e-06 -0.010020414765013672 0.028054295745135273" rpy="0 0 0"/>
-    <mass value="1.291881447401789"/>
-    <inertia ixx="0.001017" iyy="0.000798" izz="0.00122" ixy="-0.0" iyz="-3.2e-05" ixz="0.0"/>
-  </inertial>
-  <visual>
-    <origin xyz="0 0 0" rpy="0 0 0"/>
-    <geometry>
+    <inertial>
+      <origin xyz="3.5241524236579847e-09 -0.010028213246232836 0.028055691327807355" rpy="0 0 0"/>
+      <mass value="1.29137439344346"/>
+      <inertia ixx="0.001017" iyy="0.000798" izz="0.00122" ixy="-0.0" iyz="-3.2e-05" ixz="0.0"/>
+    </inertial>
+    <visual>
+      <origin xyz="0 0 0" rpy="0 0 0"/>
+      <geometry>
         <mesh filename="package://small_arm_description/meshes/base_link.stl" scale="0.001 0.001 0.001"/>
-    </geometry>
-    <material name="silver"/>
-  </visual>
-  <collision>
-    <origin xyz="0 0 0" rpy="0 0 0"/>
-    <geometry>
+      </geometry>
+      <material name="silver"/>
+    </visual>
+    <collision>
+      <origin xyz="0 0 0" rpy="0 0 0"/>
+      <geometry>
         <mesh filename="package://small_arm_description/meshes/base_link.stl" scale="0.001 0.001 0.001"/>
       </geometry>
@@ -32,19 +32,19 @@
   </link>
   <link name="link1">
-  <inertial>
-    <origin xyz="0.0005537302728879505 -3.989448908630728e-05 0.037038629210684425" rpy="0 0 0"/>
-    <mass value="0.817449728930332"/>
-    <inertia ixx="0.000383" iyy="0.000409" izz="0.00022" ixy="0.0" iyz="0.0" ixz="-3e-06"/>
-  </inertial>
-  <visual>
-    <origin xyz="0.0 -4.1e-05 -0.053" rpy="0 0 0"/>
-    <geometry>
+    <inertial>
+      <origin xyz="0.0005540343927201894 -3.987648307993698e-05 0.03705266234964923" rpy="0 0 0"/>
+      <mass value="0.8170010155014609"/>
+      <inertia ixx="0.000382" iyy="0.000409" izz="0.000219" ixy="0.0" iyz="0.0" ixz="-3e-06"/>
+    </inertial>
+    <visual>
+      <origin xyz="0.0 -4.1e-05 -0.053" rpy="0 0 0"/>
+      <geometry>
         <mesh filename="package://small_arm_description/meshes/link_1_1.stl" scale="0.001 0.001 0.001"/>
-    </geometry>
-    <material name="silver"/>
-  </visual>
-  <collision>
-    <origin xyz="0.0 -4.1e-05 -0.053" rpy="0 0 0"/>
-    <geometry>
+      </geometry>
+      <material name="silver"/>
+    </visual>
+    <collision>
+      <origin xyz="0.0 -4.1e-05 -0.053" rpy="0 0 0"/>
+      <geometry>
         <mesh filename="package://small_arm_description/meshes/link_1_1.stl" scale="0.001 0.001 0.001"/>
       </geometry>
@@ -52,19 +52,19 @@
   </link>
   <link name="link2">
-  <inertial>
-    <origin xyz="-0.024427682432744808 -0.0006951262423943992 0.09244818830678549" rpy="0 0 0"/>
-    <mass value="2.530467328750089"/>
-    <inertia ixx="0.007365" iyy="0.007836" izz="0.001385" ixy="-0.0" iyz="0.00013" ixz="-3e-05"/>
-  </inertial>
-  <visual>
-    <origin xyz="-0.0245 0.0 -0.109" rpy="0 0 0"/>
-    <geometry>
+    <inertial>
+      <origin xyz="-0.024402503506776505 -0.000948414974992276 0.08721596254239226" rpy="0 0 0"/>
+      <mass value="2.207557884875517"/>
+      <inertia ixx="0.005523" iyy="0.005928" izz="0.001196" ixy="-0.0" iyz="8.7e-05" ixz="-2.5e-05"/>
+    </inertial>
+    <visual>
+      <origin xyz="-0.0245 0.0 -0.109" rpy="0 0 0"/>
+      <geometry>
         <mesh filename="package://small_arm_description/meshes/link_2_1.stl" scale="0.001 0.001 0.001"/>
-    </geometry>
-    <material name="silver"/>
-  </visual>
-  <collision>
-    <origin xyz="-0.0245 0.0 -0.109" rpy="0 0 0"/>
-    <geometry>
+      </geometry>
+      <material name="silver"/>
+    </visual>
+    <collision>
+      <origin xyz="-0.0245 0.0 -0.109" rpy="0 0 0"/>
+      <geometry>
         <mesh filename="package://small_arm_description/meshes/link_2_1.stl" scale="0.001 0.001 0.001"/>
       </geometry>
@@ -72,19 +72,19 @@
   </link>
   <link name="link3">
-  <inertial>
-    <origin xyz="-0.02460425910708876 0.07785646945010617 0.0036503427791832466" rpy="0 0 0"/>
-    <mass value="1.5891656965493803"/>
-    <inertia ixx="0.002408" iyy="0.001132" izz="0.002797" ixy="3e-06" iyz="-5.1e-05" ixz="0.0"/>
-  </inertial>
-  <visual>
-    <origin xyz="-0.0244 -0.0 -0.279" rpy="0 0 0"/>
-    <geometry>
+    <inertial>
+      <origin xyz="-0.024604835871039465 0.06321426100068431 0.0039992416943318565" rpy="0 0 0"/>
+      <mass value="1.4545470633400195"/>
+      <inertia ixx="0.001649" iyy="0.001003" izz="0.00194" ixy="2e-06" iyz="-1.2e-05" ixz="0.0"/>
+    </inertial>
+    <visual>
+      <origin xyz="-0.0244 -0.0 -0.264" rpy="0 0 0"/>
+      <geometry>
         <mesh filename="package://small_arm_description/meshes/link_3_1.stl" scale="0.001 0.001 0.001"/>
-    </geometry>
-    <material name="silver"/>
-  </visual>
-  <collision>
-    <origin xyz="-0.0244 -0.0 -0.279" rpy="0 0 0"/>
-    <geometry>
+      </geometry>
+      <material name="silver"/>
+    </visual>
+    <collision>
+      <origin xyz="-0.0244 -0.0 -0.264" rpy="0 0 0"/>
+      <geometry>
         <mesh filename="package://small_arm_description/meshes/link_3_1.stl" scale="0.001 0.001 0.001"/>
       </geometry>
@@ -92,19 +92,19 @@
   </link>
   <link name="link4">
-  <inertial>
-    <origin xyz="0.0005678122855020656 0.028502036892318075 0.00010812835093654272" rpy="0 0 0"/>
-    <mass value="0.4500719035752892"/>
-    <inertia ixx="0.000146" iyy="8.3e-05" izz="0.000143" ixy="-1e-06" iyz="-0.0" ixz="-0.0"/>
-  </inertial>
-  <visual>
-    <origin xyz="0.0003 -0.121766 -0.280316" rpy="0 0 0"/>
-    <geometry>
+    <inertial>
+      <origin xyz="0.0005772929478554495 0.02874769471007499 0.00014670041370268283" rpy="0 0 0"/>
+      <mass value="0.4457408919666805"/>
+      <inertia ixx="0.000144" iyy="8.2e-05" izz="0.00014" ixy="-1e-06" iyz="-0.0" ixz="-0.0"/>
+    </inertial>
+    <visual>
+      <origin xyz="0.0003 -0.100766 -0.265316" rpy="0 0 0"/>
+      <geometry>
         <mesh filename="package://small_arm_description/meshes/link_4_1.stl" scale="0.001 0.001 0.001"/>
-    </geometry>
-    <material name="silver"/>
-  </visual>
-  <collision>
-    <origin xyz="0.0003 -0.121766 -0.280316" rpy="0 0 0"/>
-    <geometry>
+      </geometry>
+      <material name="silver"/>
+    </visual>
+    <collision>
+      <origin xyz="0.0003 -0.100766 -0.265316" rpy="0 0 0"/>
+      <geometry>
         <mesh filename="package://small_arm_description/meshes/link_4_1.stl" scale="0.001 0.001 0.001"/>
       </geometry>
@@ -112,19 +112,19 @@
   </link>
   <link name="link5">
-  <inertial>
-    <origin xyz="-0.019068054583883113 0.009694576419165046 -0.04274059819483081" rpy="0 0 0"/>
-    <mass value="1.0859764685043407"/>
-    <inertia ixx="0.000829" iyy="0.00064" izz="0.000658" ixy="-0.0" iyz="-0.0001" ixz="-0.0"/>
-  </inertial>
-  <visual>
-    <origin xyz="-0.0187 -0.165647 -0.280441" rpy="0 0 0"/>
-    <geometry>
+    <inertial>
+      <origin xyz="-0.019082924173376172 0.006958151104480087 -0.04482191950153944" rpy="0 0 0"/>
+      <mass value="0.9868678983343436"/>
+      <inertia ixx="0.000651" iyy="0.000558" izz="0.000526" ixy="0.0" iyz="-1.2e-05" ixz="0.0"/>
+    </inertial>
+    <visual>
+      <origin xyz="-0.0187 -0.144647 -0.265441" rpy="0 0 0"/>
+      <geometry>
         <mesh filename="package://small_arm_description/meshes/link_5_1.stl" scale="0.001 0.001 0.001"/>
-    </geometry>
-    <material name="silver"/>
-  </visual>
-  <collision>
-    <origin xyz="-0.0187 -0.165647 -0.280441" rpy="0 0 0"/>
-    <geometry>
+      </geometry>
+      <material name="silver"/>
+    </visual>
+    <collision>
+      <origin xyz="-0.0187 -0.144647 -0.265441" rpy="0 0 0"/>
+      <geometry>
         <mesh filename="package://small_arm_description/meshes/link_5_1.stl" scale="0.001 0.001 0.001"/>
       </geometry>
@@ -132,19 +132,19 @@
   </link>
   <link name="link6">
-  <inertial>
-    <origin xyz="0.004492294331015427 0.0003709408309400253 -0.019015271355907637" rpy="0 0 0"/>
-    <mass value="0.5127274279729177"/>
-    <inertia ixx="9.5e-05" iyy="0.000226" izz="0.000235" ixy="-1e-06" iyz="0.0" ixz="1e-06"/>
-  </inertial>
-  <visual>
-    <origin xyz="0.0004 -0.165647 -0.205922" rpy="0 0 0"/>
-    <geometry>
+    <inertial>
+      <origin xyz="0.004698639386755362 0.0003750363685992575 -0.018998646992087587" rpy="0 0 0"/>
+      <mass value="0.5087647252977904"/>
+      <inertia ixx="9.4e-05" iyy="0.000223" izz="0.000231" ixy="-1e-06" iyz="0.0" ixz="1e-06"/>
+    </inertial>
+    <visual>
+      <origin xyz="0.0004 -0.144647 -0.190922" rpy="0 0 0"/>
+      <geometry>
         <mesh filename="package://small_arm_description/meshes/Claw_base_1.stl" scale="0.001 0.001 0.001"/>
-    </geometry>
-    <material name="silver"/>
-  </visual>
-  <collision>
-    <origin xyz="0.0004 -0.165647 -0.205922" rpy="0 0 0"/>
-    <geometry>
+      </geometry>
+      <material name="silver"/>
+    </visual>
+    <collision>
+      <origin xyz="0.0004 -0.144647 -0.190922" rpy="0 0 0"/>
+      <geometry>
         <mesh filename="package://small_arm_description/meshes/Claw_base_1.stl" scale="0.001 0.001 0.001"/>
       </geometry>
@@ -152,19 +152,19 @@
   </link>
   <link name="gripper_link1">
-  <inertial>
-    <origin xyz="0.009553177578958301 -0.019099491341480757 -0.027462032562735744" rpy="0 0 0"/>
-    <mass value="0.3481919018430052"/>
-    <inertia ixx="0.000338" iyy="0.000245" izz="0.000155" ixy="0.0" iyz="-0.0" ixz="2.6e-05"/>
-  </inertial>
-  <visual>
-    <origin xyz="-0.0216 -0.184647 -0.184772" rpy="0 0 0"/>
-    <geometry>
+    <inertial>
+      <origin xyz="0.008617592547608088 -0.019099487462018033 -0.018966140525552982" rpy="0 0 0"/>
+      <mass value="0.27120735685123026"/>
+      <inertia ixx="0.000219" iyy="0.000142" izz="0.000135" ixy="0.0" iyz="-0.0" ixz="2e-05"/>
+    </inertial>
+    <visual>
+      <origin xyz="-0.0216 -0.163647 -0.169772" rpy="0 0 0"/>
+      <geometry>
         <mesh filename="package://small_arm_description/meshes/Claw_1_1.stl" scale="0.001 0.001 0.001"/>
-    </geometry>
-    <material name="silver"/>
-  </visual>
-  <collision>
-    <origin xyz="-0.0216 -0.184647 -0.184772" rpy="0 0 0"/>
-    <geometry>
+      </geometry>
+      <material name="silver"/>
+    </visual>
+    <collision>
+      <origin xyz="-0.0216 -0.163647 -0.169772" rpy="0 0 0"/>
+      <geometry>
         <mesh filename="package://small_arm_description/meshes/Claw_1_1.stl" scale="0.001 0.001 0.001"/>
       </geometry>
@@ -172,19 +172,19 @@
   </link>
 <link name="gripper_link2">
-  <inertial>
-    <origin xyz="-0.008862773747378604 -0.01908264305352636 -0.025794573876087107" rpy="0 0 0"/>
-    <mass value="0.3632084794432327"/>
-    <inertia ixx="0.000361" iyy="0.000263" izz="0.000164" ixy="0.0" iyz="0.0" ixz="-3.1e-05"/>
-  </inertial>
-  <visual>
-    <origin xyz="0.0224 -0.184582 -0.184772" rpy="0 0 0"/>
-    <geometry>
+    <inertial>
+      <origin xyz="-0.0077905784072223 -0.019078107759134433 -0.01729592412140632" rpy="0 0 0"/>
+      <mass value="0.2862239344986947"/>
+      <inertia ixx="0.000234" iyy="0.00015" izz="0.000143" ixy="0.0" iyz="0.0" ixz="-2.3e-05"/>
+    </inertial>
+    <visual>
+      <origin xyz="0.0224 -0.163582 -0.169772" rpy="0 0 0"/>
+      <geometry>
         <mesh filename="package://small_arm_description/meshes/Claw_2_1.stl" scale="0.001 0.001 0.001"/>
-    </geometry>
-    <material name="silver"/>
-  </visual>
-  <collision>
-    <origin xyz="0.0224 -0.184582 -0.184772" rpy="0 0 0"/>
-    <geometry>
+      </geometry>
+      <material name="silver"/>
+    </visual>
+    <collision>
+      <origin xyz="0.0224 -0.163582 -0.169772" rpy="0 0 0"/>
+      <geometry>
         <mesh filename="package://small_arm_description/meshes/Claw_2_1.stl" scale="0.001 0.001 0.001"/>
       </geometry>
@@ -192,19 +192,19 @@
   </link>
   <link name="camera_link">
-  <inertial>
-    <origin xyz="-0.022501861739521612 -4.8500070798096484e-05 -0.012169837448304244" rpy="0 0 0"/>
-    <mass value="0.37837987609307205"/>
-    <inertia ixx="3.5e-05" iyy="0.00024" izz="0.000238" ixy="-0.0" iyz="-0.0" ixz="0.0"/>
-  </inertial>
-  <visual>
-    <origin xyz="-0.0222 -0.225439 -0.254372" rpy="0 0 0"/>
-    <geometry>
+    <inertial>
+      <origin xyz="-1.8617389460899472e-06 -0.008048500132108033 -0.012169837419856416" rpy="0 0 0"/>
+      <mass value="0.3783798760930714"/>
+      <inertia ixx="3.5e-05" iyy="0.00024" izz="0.000238" ixy="-0.0" iyz="-0.0" ixz="0.0"/>
+    </inertial>
+    <visual>
+      <origin xyz="0.0004 -0.202439 -0.219372" rpy="0 0 0"/>
+      <geometry>
         <mesh filename="package://small_arm_description/meshes/Camera_1.stl" scale="0.001 0.001 0.001"/>
-    </geometry>
-    <material name="silver"/>
-  </visual>
-  <collision>
-    <origin xyz="-0.0222 -0.225439 -0.254372" rpy="0 0 0"/>
-    <geometry>
+      </geometry>
+      <material name="silver"/>
+    </visual>
+    <collision>
+      <origin xyz="0.0004 -0.202439 -0.219372" rpy="0 0 0"/>
+      <geometry>
         <mesh filename="package://small_arm_description/meshes/Camera_1.stl" scale="0.001 0.001 0.001"/>
       </geometry>
@@ -234,5 +234,5 @@
   </joint>
   <joint name="joint3" type="revolute">
-    <origin xyz="-0.0001 0.0 0.17" rpy="0 0 0"/>
+    <origin xyz="-0.0001 0.0 0.155" rpy="0 0 0"/>
     <parent link="link2"/>
     <child link="link3"/>
@@ -245,8 +245,8 @@
   </joint>
   <joint name="joint4" type="revolute">
-    <origin xyz="-0.0247 0.121766 0.001316" rpy="0 0 0"/>
+    <origin xyz="-0.0247 0.100766 0.001316" rpy="0 0 0"/>
     <parent link="link3"/>
     <child link="link4"/>
-    <axis xyz="-0.0 1.0 -0.0"/>
+    <axis xyz="-0.0 -1.0 -0.0"/>
     <limit
       lower="-3.14"
@@ -267,5 +267,5 @@
   </joint>
   <joint name="joint6" type="revolute">
-    <origin xyz="-0.0191 0.0 -0.074519" rpy="0 0 0"/>
+    <origin xyz="-0.019 0.0 -0.069019" rpy="0 0 0"/>
     <parent link="link5"/>
     <child link="link6"/>
@@ -306,5 +306,5 @@
   </joint> -->
   <joint name="camera_fixed" type="fixed">
-    <origin xyz="0.0035 0.059792 -0.026069" rpy="0 0 0"/>
+    <origin xyz="-0.0191 0.057792 -0.046069" rpy="0 0 0"/>
     <parent link="link5"/>
     <child link="camera_link"/>

File: small_arm_description/urdf/small_arm.ros2_control.xacro (robot description, xacro)
@@ -7,5 +7,5 @@
         <param name="usb_port">/dev/ttyUSB0</param>
         <param name="baud_rate">115200</param>
-        <param name="use_dummy">false</param>
+        <param name="use_dummy">true</param>
       </hardware>
       <joint name="joint1">

File: small_arm_description/urdf/small_arm.urdf.xacro (robot description, xacro)
@@ -2,9 +2,9 @@
 <robot name="small_arm" xmlns:xacro="http://ros.org/wiki/xacro">
   <xacro:include filename="$(find small_arm_description)/urdf/small_arm.xacro" />
-  <xacro:include filename="$(find small_arm_description)/urdf/small_arm.ros2_control.xacro" />
+  <!-- <xacro:include filename="$(find small_arm_description)/urdf/small_arm.ros2_control.xacro" /> -->
   <link name="world"/>
   <xacro:small_arm parent="world">
     <origin xyz="0 0 0" rpy="0 0 0" />
   </xacro:small_arm>
-  <xacro:small_arm_ros2_control name="small_arm_ros2_control" />
+  <!-- <xacro:small_arm_ros2_control name="small_arm_ros2_control" /> -->
 </robot>

File: small_arm_moveit_config/config/small_arm.ros2_control.xacro (robot description, xacro)
@@ -12,5 +12,5 @@
                     <param name="usb_port">/dev/ttyUSB0</param>
                     <param name="baud_rate">115200</param>
-                    <param name="use_dummy">true</param>
+                    <param name="use_dummy">false</param>
                 </xacro:if>
             </hardware>
